File: CtrlKeys.kicad_sch (KiCad schematic)
At the start: 0 parts

Commit message: Wired basic schematic (without battery mechanics)
Parts:
- added C1, C2: 10 uF, Capacitor_SMD:C_0603_1608Metric_Pad1.08x0.95mm_HandSolder, symbol Device:C_Small
- added D1, D2, D3, D4, D5, D6, D7, D8: WS2812B, LED_SMD:LED_WS2812B_PLCC4_5.0x5.0mm_P3.2mm, symbol LED:WS2812B
- added J1: Connector_USB_C_Receptacle_USB2.0, symbol USB-C-USB-2.0-cache:Connector_USB_C_Receptacle_USB2.0
- added J2: DBG_HEADER, Connector_PinSocket_2.54mm:PinSocket_1x05_P2.54mm_Vertical, symbol Connector:Conn_01x05_Pin
- added L1: 3.9 uH, Inductor_SMD:L_0603_1608Metric_Pad1.05x0.95mm_HandSolder, symbol Device:L_Small
- added R1, R2: 5.1k, Resistor_SMD:R_0402_1005Metric_Pad0.72x0.64mm_HandSolder, symbol Device:R
- added R3: 100k, Resistor_SMD:R_0402_1005Metric_Pad0.72x0.64mm_HandSolder, symbol Device:R
- added SW1, SW2, SW3, SW4, SW5, SW6: SW_Push, Button_Switch_Keyboard:SW_Cherry_MX_1.00u_PCB, symbol Switch:SW_Push
- added SW7: BOOT, Button_Switch_SMD:SW_Push_1P1T_NO_CK_KMR2, symbol Switch:SW_Push
- added SW8: RST, Button_Switch_SMD:SW_Push_1P1T_NO_CK_KMR2, symbol Switch:SW_Push
- added U1: ESP32-S3-WROOM-1, RF_Module:ESP32-S3-WROOM-1, symbol RF_Module:ESP32-S3-WROOM-1
- added U2: AP63203WU, Package_TO_SOT_SMD:TSOT-23-6, symbol Regulator_Switching:AP63203WU
- added U3: SN74LVC1T45DBV, Package_TO_SOT_SMD:SOT-23-6_Handsoldering, symbol Logic_LevelTranslator:SN74LVC1T45DBV
Connections:
- new net: J1.B5 (CC2), R1.1
- new net: SW1.1, U1.5 (IO5)
- new net: C2.1, U2.6 (BST)
- new net: C2.2, L1.1, U2.5 (SW)
- new net: J1.A5 (CC1), R2.1
- new net: J1.A6 (D+), J1.B6 (D+), U1.14 (USB_D+)
- new net: J1.A7 (D-), J1.B7 (D-), U1.13 (USB_D-)
- new net: D5.2 (DOUT), D6.4 (DIN)
- new net: D4.2 (DOUT), D5.4 (DIN)
- new net: SW4.1, U1.4 (IO4)
- new net: D3.2 (DOUT), D4.4 (DIN)
- new net: J2.2 (Pin_2), U1.37 (TXD0)
- new net: J2.4 (Pin_4), U1.36 (RXD0)
- new net: D2.2 (DOUT), D3.4 (DIN)
- new net: D7.2 (DOUT), D8.4 (DIN)
- new net: D6.2 (DOUT), D7.4 (DIN)
- new net: SW6.1, U1.12 (IO8)
- new net: SW3.1, U1.17 (IO9)
- new net: SW7.1, U1.27 (IO0)
- new net: R3.2, SW8.1, U1.3 (EN)
- new net: U1.39 (IO1), U3.3 (A)
- new net: SW5.1, U1.6 (IO6)
- new net: SW2.1, U1.7 (IO7)
- new net: D1.2 (DOUT), D2.4 (DIN)
- new net: D1.4 (DIN), U3.4 (B)
- new net +3.3V: J2.1 (Pin_1), L1.2, R3.1, U1.2 (3V3), U2.1 (FB), U3.1 (VCCA), U3.5 (DIR)
- new net +5V: C1.1, D1.1 (VDD), D2.1 (VDD), D3.1 (VDD), D4.1 (VDD), D5.1 (VDD), D6.1 (VDD), D7.1 (VDD), D8.1 (VDD), J1.A4 (VBUS), J1.A9 (VBUS), J1.B4 (VBUS), J1.B9 (VBUS), J2.5 (Pin_5), U2.2 (EN), U2.3 (IN), U3.6 (VCCB)
- new net GND: C1.2, D1.3 (VSS), D2.3 (VSS), D3.3 (VSS), D4.3 (VSS), D5.3 (VSS), D6.3 (VSS), D7.3 (VSS), D8.3 (VSS), J1.A1 (GND), J1.A12 (GND), J1.B1 (GND), J1.B12 (GND), J1.S1 (SHIELD), J2.3 (Pin_3), R1.2, R2.2, SW1.2, SW2.2, SW3.2, SW4.2, SW5.2, SW6.2, SW7.2, SW8.2, U1.1 (GND), U1.40 (GND), U1.41 (GND), U2.4 (GND), U3.2 (GND)
- no-connect marks 0 -> 2
